File: FCSat_dual/FCSat_dual.kicad_pcb (KiCad board)
At the start: 2 copper layers, 93 x 93 mm, 189 parts, among them J1 Conn_01x02_Pin, J10 Conn_01x04_Pin, J11 Conn_01x04_Pin, J12 Conn_02x03_Odd_Even, J2 Conn_01x04_Pin, J3 Y!:105162-0001 SD, J4 Conn_Coaxial, J5 L834-1G1T-91, J6 105162-0001, J7 Conn_01x04_Pin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

Commit message: added attiny, and changes in layout
Parts:
- removed C57, C60: 22uF, Capacitor_SMD:C_0805_2012Metric_Pad1.18x1.45mm_HandSolder
- removed USB_C_ESP3: USB_C, Connector_USB:USB_C_Receptacle_G-Switch_GT-USB-7010ASV
- added C54: 2.2nF, Capacitor_SMD:C_0402_1005Metric_Pad0.74x0.62mm_HandSolder, F.Cu at (177.2, 127.4)
- added C55: 100n, Capacitor_SMD:C_0603_1608Metric, F.Cu at (173.6, 127.7)
- added USB_C_ESP2: USB_C, Connector_USB:USB_C_Receptacle_G-Switch_GT-USB-7010ASV, F.Cu at (177.4, 121.8)
- C1: value 10p -> 20pF
- C20: value 100n -> 4.7uF
- C23: value 2.2uF -> 100n; footprint Capacitor_SMD:C_0402_1005Metric_Pad0.74x0.62mm_HandSolder -> Capacitor_SMD:C_0603_1608Metric
- C24: value 2.2uF -> 10u; footprint Capacitor_SMD:C_0402_1005Metric_Pad0.74x0.62mm_HandSolder -> Capacitor_SMD:C_0603_1608Metric
- C26, C27: value 100n -> 10p
- C28, C29, C34: value 100n -> 22uF; footprint Capacitor_SMD:C_0603_1608Metric -> Capacitor_SMD:C_0805_2012Metric_Pad1.18x1.45mm_HandSolder
- C3: value 10p -> 4.7uF
- C31: value 2.2nF -> 100n; footprint Capacitor_SMD:C_0402_1005Metric_Pad0.74x0.62mm_HandSolder -> Capacitor_SMD:C_0603_1608Metric
- C32, C43: value 100n -> 10u
- C33: value 10nF -> 22uF; footprint Capacitor_SMD:C_0402_1005Metric_Pad0.74x0.62mm_HandSolder -> Capacitor_SMD:C_0805_2012Metric_Pad1.18x1.45mm_HandSolder
- C35: value 10u -> 10p
- C36: value 22uF -> 10p; footprint Capacitor_SMD:C_0805_2012Metric_Pad1.18x1.45mm_HandSolder -> Capacitor_SMD:C_0603_1608Metric
- C37: value 22uF -> 10u; footprint Capacitor_SMD:C_0805_2012Metric_Pad1.18x1.45mm_HandSolder -> Capacitor_SMD:C_0603_1608Metric
- C38: value 10p -> 100n
- C39: value 10p -> 470p
- C4: value 20pF -> 2.2uF; footprint Capacitor_SMD:C_0603_1608Metric -> Capacitor_SMD:C_0402_1005Metric_Pad0.74x0.62mm_HandSolder
- C40, C46, C52: value 10u -> 100n
- C41: value 100n -> 1u
- C42: value 470p -> 100n
- C44: value 1u -> 0.022u
- C45: value 100n -> 0.022u
- C47, C48: value 0.022u -> 100n
- C49: value 100n -> 10nF; footprint Capacitor_SMD:C_0603_1608Metric -> Capacitor_SMD:C_0402_1005Metric_Pad0.74x0.62mm_HandSolder
- C7: value 4.7uF -> 2.2uF; footprint Capacitor_SMD:C_0603_1608Metric -> Capacitor_SMD:C_0402_1005Metric_Pad0.74x0.62mm_HandSolder
- C8: value 4.7uF -> 100n
- D1: value led -> 0402ESDA-MLP1; footprint LED_SMD:LED_0603_1608Metric -> Diode_SMD:D_0402_1005Metric_Pad0.77x0.64mm_HandSolder
- D10, D11: value BAV99 -> led; footprint Package_TO_SOT_SMD:SOT-23 -> LED_SMD:LED_0603_1608Metric
- D12: value 0402ESDA-MLP1 -> led; footprint Diode_SMD:D_0402_1005Metric_Pad0.77x0.64mm_HandSolder -> LED_SMD:LED_0603_1608Metric
- D13, D14: value led -> GREEN LED
- D15: value GREEN LED -> led
- D3: value 0402ESDA-MLP1 -> BAT54; footprint Diode_SMD:D_0402_1005Metric_Pad0.77x0.64mm_HandSolder -> Package_TO_SOT_SMD:SOT-23
- D5: value GREEN LED -> 0402ESDA-MLP1; footprint LED_SMD:LED_0603_1608Metric -> Diode_SMD:D_0402_1005Metric_Pad0.77x0.64mm_HandSolder
- D6: value led -> BAV99; footprint LED_SMD:LED_0603_1608Metric -> Package_TO_SOT_SMD:SOT-23
- D7: value BAT54 -> BAV99
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Connections:
- 1.8vReg1 pad 1: 1CAM1_IO0 -> HDMI_HPD_N_1V8
- 1.8vReg2 pad 1: 1CAM1_IO0 -> HDMI_HPD_N_1V8
- Accel1 pad 1: 1CAM1_IO0 -> HDMI_HPD_N_1V8
- Accel1 pad 11: 1CAM1_IO0 -> HDMI_HPD_N_1V8
- Accel1 pad 18: 1CAM1_IO0 -> HDMI_HPD_N_1V8
- Alt1 pad 2: 1CAM1_IO0 -> HDMI_HPD_N_1V8
- Alt1 pad 3: 1CAM1_IO0 -> HDMI_HPD_N_1V8
- BATCharge1 pad 1: 1CAM1_IO0 -> HDMI_HPD_N_1V8
- BATCharge1 pad 3: 1CAM1_IO0 -> HDMI_HPD_N_1V8
- BATCharge2 pad 1: 1CAM1_IO0 -> HDMI_HPD_N_1V8
- BATCharge2 pad 3: 1CAM1_IO0 -> HDMI_HPD_N_1V8
- BT1 pad 2: 1CAM1_IO0 -> HDMI_HPD_N_1V8
- BatProt1 pad 4: 1CAM1_IO0 -> HDMI_HPD_N_1V8
- BatProt2 pad 4: 1CAM1_IO0 -> HDMI_HPD_N_1V8
- C1 pad 1: 1CAM1_IO0 -> Net-(MainMCU1-PH0)
- C1 pad 2: Net-(MainMCU1-PC15) -> HDMI_HPD_N_1V8
- C10 pad 2: 1CAM1_IO0 -> HDMI_HPD_N_1V8
- C11 pad 2: 1CAM1_IO0 -> HDMI_HPD_N_1V8
- C12 pad 2: 1CAM1_IO0 -> HDMI_HPD_N_1V8
- C13 pad 2: 1CAM1_IO0 -> HDMI_HPD_N_1V8
- C14 pad 2: 1CAM1_IO0 -> HDMI_HPD_N_1V8
- C15 pad 2: 1CAM1_IO0 -> HDMI_HPD_N_1V8
- C16 pad 2: 1CAM1_IO0 -> HDMI_HPD_N_1V8
- C17 pad 1: +3V3 -> HDMI_HPD_N_1V8
- C17 pad 2: 1CAM1_IO0 -> Net-(MainMCU1-VDD33_USB)
- C18 pad 1: +3V3 -> HDMI_HPD_N_1V8
- C18 pad 2: 1CAM1_IO0 -> Net-(MainMCU1-VDD50_USB)
- C19 pad 2: 1CAM1_IO0 -> HDMI_HPD_N_1V8
- C2 pad 1: Net-(MainMCU1-PH0) -> Net-(MainMCU1-PH1)
- C2 pad 2: 1CAM1_IO0 -> HDMI_HPD_N_1V8
- C20 pad 1: +3V3 -> HDMI_HPD_N_1V8
- C20 pad 2: 1CAM1_IO0 -> Net-(C20-Pad2)
- C21 pad 1: 1CAM1_IO0 -> +3V3
- C21 pad 2: Net-(MainMCU1-VDD33_USB) -> HDMI_HPD_N_1V8
- C22 pad 1: 1CAM1_IO0 -> HDMI_HPD_N_1V8
- C22 pad 2: Net-(MainMCU1-VDD50_USB) -> Net-(BatProt1-BAT)
- C23 pad 1: 1CAM1_IO0 -> +3V3
- C23 pad 2: Net-(C23-Pad2) -> HDMI_HPD_N_1V8
- C24 pad 1: 1CAM1_IO0 -> Net-(1.8vReg1-VI)
- C24 pad 2: Net-(MainMCU1-VCAPDSI) -> Net-(PowerMosfet1-S2)
- C25 pad 1: 1CAM1_IO0 -> +3V3
- C25 pad 2: Net-(GPS1-VCC) -> HDMI_HPD_N_1V8
- C26 pad 1: +3V3 -> HDMI_HPD_N_1V8
- C26 pad 2: 1CAM1_IO0 -> Net-(MainMCU1-PC14)
- C27 pad 1: 1CAM1_IO0 -> HDMI_HPD_N_1V8
- C27 pad 2: +3V3 -> Net-(MainMCU1-PC15)
- C28 pad 1: 1CAM1_IO0 -> +1V8
- C28 pad 2: +3V3 -> HDMI_HPD_N_1V8
- C29 pad 1: 1CAM1_IO0 -> +3.3V
- C29 pad 2: +3V3 -> HDMI_HPD_N_1V8
- C3 pad 1: 1CAM1_IO0 -> +3V3
- C3 pad 2: Net-(MainMCU1-PC14) -> HDMI_HPD_N_1V8
- C30 pad 1: 1CAM1_IO0 -> Net-(D3-K)
- C30 pad 2: +3V3 -> HDMI_HPD_N_1V8
- C31 pad 1: Net-(Accel1-CPOUT) -> HDMI_HPD_N_1V8
- C31 pad 2: 1CAM1_IO0 -> Net-(BatProt2-BAT)
- C32 pad 1: 1CAM1_IO0 -> Net-(1.8vReg2-VI)
- C32 pad 2: Net-(Accel1-REGOUT) -> Net-(PowerMosfet2-S2)
- C33 pad 1: Net-(C33-Pad1) -> VCC
- C33 pad 2: 1CAM1_IO0 -> HDMI_HPD_N_1V8
- C34 pad 1: 1CAM1_IO0 -> +3.3VA
- C34 pad 2: Net-(BatProt1-BAT) -> HDMI_HPD_N_1V8
- C35 pad 1: Net-(1.8vReg1-VI) -> HDMI_HPD_N_1V8
- C35 pad 2: Net-(PowerMosfet1-S2) -> Net-(U4-XTAL1/CLKIN)
- C36 pad 1: +1V8 -> HDMI_HPD_N_1V8
- C36 pad 2: 1CAM1_IO0 -> Net-(U4-XTAL2)
- C37 pad 1: +3.3V -> +3.3VA
- C37 pad 2: 1CAM1_IO0 -> HDMI_HPD_N_1V8
- C38 pad 1: 1CAM1_IO0 -> +3.3VA
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