File: FCSat_dual/FCSat_dual.kicad_sch (KiCad schematic)
At the start: 189 parts, among them J1 Conn_01x02_Pin, J1 Y!:105162-0001 SD, J10 Conn_01x04_Pin, J11 Conn_01x04_Pin, J12 Conn_02x03_Odd_Even, J2 Conn_01x04_Pin, J2 Conn_Coaxial, J3 L834-1G1T-91, J4 105162-0001, J7 Conn_01x04_Pin, J8 2001-1-2-21-00-BK, J9 Conn_01x04_Pin, P1 CAM1, P2 CAM1, P3 CONN_02X20, P4 CONN_02X20, Q1 BCV27, Q2 2N7002P.215, Q3 2N7002P.215, Q4 2N7002P.215, SW3 SW_Push, SW3 SW_Push_SPDT, U2 IS25LP032D, U9 LAN8742A, Y1 32.768K, Y2 8MHz, Y3 25M

Commit message: added attiny, and changes in layout
Parts:
- renumbered 1.8vReg1 to 1.8vReg?, Accel1 to Accel?, Alt1 to Alt?, BAT1 to BAT?, BATCharge1 to BATCharge?, BT1 to BT?, BatProt1 to BatProt?, C2 to C?, C5 to C?, C4 to C?, C33 to C?, C9 to C?, C3 to C?, C35 to C?, C44 to C?, C41 to C?, C32 to C?, C31 to C?, C14 to C?, C43 to C?, C46 to C?, C30 to C?, C25 to C?, C10 to C?, C38 to C?, C12 to C?, C11 to C?, C29 to C?, C7 to C?, C8 to C?, C39 to C?, C47 to C?, C36 to C?, C45 to C?, C6 to C?, C34 to C?, C40 to C?, C37 to C?, D15 to D13, D5 to D14, D7 to D3, D8 to D6, D9 to D7, D10 to D8, D11 to D9, D1 to D?, D9 to D?, D4 to D?, D7 to D?, D3 to D?, D6 to D?, FB1 to FB?, GPS1 to GPS?, IMU1 to IMU?, J2 to J1, J1 to J2, J8 to J3, J12 to J4, J7 to J5, J9 to J6, J10 to J7, J11 to J9, J4 to J?, J1 to J?, J2 to J?, J3 to J?, L2 to L?, L1 to L?, L5 to L?, LoRaWan1 to LoRaWan?, Magnetometer1 to Magnetometer?, P4 to P3, P3 to P4, PowerMosfet2 to PowerMosfet?, Q2 to Q1, Q4 to Q2, Q1 to Q?, R44 to R23, R59 to R28, R60 to R29, R41 to R30, R42 to R31, R2 to R?, R26 to R?, R16 to R?, R25 to R?, R9 to R?, R7 to R?, R32 to R?, R15 to R?, R6 to R?, R5 to R?, R28 to R?, R8 to R?, R4 to R?, R12 to R?, R14 to R?, R3 to R?, R29 to R?, R30 to R?, R27 to R?, R22 to R?, R18 to R?, R33 to R?, R24 to R?, R19 to R?, R31 to R?, R34 to R?, R13 to R?, R17 to R?, SW3 to SW?, U2 to U1, U3 to U2, U4 to U3, U9 to U?, U2 to U?, USB_C_ESP1 to USB_C_ESP?, VoltReg1 to VoltReg?, Y3 to Y?, Y1 to Y?, Y2 to Y?

Commit message: new update
Parts:
- removed 1.8vReg?: LD1117S18TR_SOT223, Package_TO_SOT_SMD:SOT-223-3_TabPin2, symbol Regulator_Linear:LD1117S18TR_SOT223
- removed BT?: Battery, Connector_PinSocket_2.54mm:PinSocket_1x02_P2.54mm_Vertical, symbol Device:Battery
- removed C? (x2): 22uF, Capacitor_SMD:C_0805_2012Metric_Pad1.18x1.45mm_HandSolder, symbol Device:C_Small
- removed J1, J5, J6, J7, J9: Conn_01x04_Pin, Connector_PinSocket_2.54mm:PinSocket_1x04_P2.54mm_Vertical, symbol Connector:Conn_01x04_Pin
- removed J2: Conn_01x02_Pin, Connector_PinSocket_2.54mm:PinSocket_1x02_P2.54mm_Vertical, symbol Connector:Conn_01x02_Pin
- removed SW?: SW_Push_SPDT, Connector_PinSocket_2.54mm:PinSocket_1x03_P2.54mm_Vertical, symbol Switch:SW_Push_SPDT
- removed VoltReg?: AMS1117CD-3.3, Package_TO_SOT_SMD:SOT-223-3_TabPin2, symbol Regulator_Linear:AMS1117CD-3.3
- added 1.8vReg1: LD1117S18TR_SOT223, Package_TO_SOT_SMD:SOT-223-3_TabPin2, symbol Regulator_Linear:LD1117S18TR_SOT223
- added C3 (x2): 22uF, Capacitor_SMD:C_0805_2012Metric_Pad1.18x1.45mm_HandSolder, symbol Device:C_Small
- added C30 (x6): 15uF, Capacitor_SMD:C_0603_1608Metric, symbol Device:C_Small
- added C30 (x4): 180uF, Capacitor_SMD:C_0603_1608Metric, symbol Device:C_Small
- added C30 (x2): 100nF, Capacitor_SMD:C_0603_1608Metric, symbol Device:C_Small
- added C30 (x2): 1nF, Capacitor_SMD:C_0603_1608Metric, symbol Device:C_Small
- added C30 (x2): .47uF, Capacitor_SMD:C_0603_1608Metric, symbol Device:C_Small
- added D16, D17: PMEG100V060ELPDZ, Package_TO_SOT_SMD:TO-277B, symbol Device:D_Schottky_Small
- added J10, J11, J13, J14, J15, J16, J7, J9: Conn_01x03_Pin, Connector_PinHeader_2.54mm:PinHeader_1x03_P2.54mm_Vertical, symbol Connector:Conn_01x03_Pin
- added L1 (x2): 22uH, Inductor_SMD:L_0603_1608Metric, symbol Device:L_Small
- added R7 (x2): 5.6k, Resistor_SMD:R_0402_1005Metric, symbol Device:R
- added R9: NC, Resistor_SMD:R_0402_1005Metric, symbol Device:R
- added R9: 0, Resistor_SMD:R_0402_1005Metric, symbol Device:R
- added U6, U7: LM2672M-5.0, Package_TO_SOT_SMD:TO-263-7_TabPin8, symbol Regulator_Switching:LM2672M-5.0
- added VoltReg1: AMS1117CD-3.3, Package_TO_SOT_SMD:SOT-223-3_TabPin2, symbol Regulator_Linear:AMS1117CD-3.3
- BAT1: renamed from BAT?; footprint Connector_PinHeader_2.54mm:PinHeader_1x02_P2.54mm_Vertical -> Y!:AMASS_XT60PW-M
- R12, R32, R33, R34: renamed from R?; value 49.9R -> 50R
- gave numbers to parts that had none: 90
- renumbered D8 to D10, D9 to D11, D13 to D15, D14 to D5, D3 to D7, D6 to D8, D7 to D9, J4 to J12, J3 to J8, P4 to P3, P3 to P4, Q1 to Q2, Q2 to Q4, R30 to R41, R31 to R42, R23 to R44, R28 to R59, R29 to R60, U1 to U2, U2 to U3, U3 to U4
Connections:
- net +3V3 is gone; now on net +3.3V: Accel1.13 (VDD), Alt1.1 (VDD), C14.1, C2.1, C2.1, C2.2, C2.2, C2.2, C2.2, C3.1, C39.1, C4.1, C40.1, C41.1, C43.1, C44.1, C45.1, C46.1, C47.1, C5.1, C6.1, D7.2 (A), FB1.1, IMU1.5 (VDDIO), IMU1.8 (VDD), J1.4 (VDD), J4.4 (VDD), L1.2, LoRaWan1.20 (VDD), Magnetometer1.13 (DVDD), Magnetometer1.2 (AVDD), Magnetometer1.7 (VPP), MainMCU1.113 (VDD), MainMCU1.126 (VDD), MainMCU1.13 (VDD), MainMCU1.136 (VDD), MainMCU1.152 (VDD), MainMCU1.160 (VDD), MainMCU1.174 (PDR_ON), MainMCU1.176 (VDD), MainMCU1.25 (VDD), MainMCU1.39 (VREF+), MainMCU1.44 (VDD), MainMCU1.48 (VDD), MainMCU1.65 (VDD), MainMCU1.7 (VDD), MainMCU1.71 (VDD), MainMCU1.84 (VDD), MainMCU1.92 (VDD), MainMCU1.99 (VDD), R2.2, R2.2, R27.1, R28.1, R29.1, R30.1, R31.1, SW3.1, U2.8 (VCC)
- net FlVCC is gone; now on net +1V8: D6.2 (A)
- net GPIO14 is gone; now on net PC_TX: P3.8 (P8)
- net GPIO15 is gone; now on net PC_RX: P3.10 (P10)
- net VBus is gone; now on net Vbus: D4.2 (A)
- net +3.3V: now also MainMCU1.8 (VBAT)
- net +3.3VA: now also C3.1, J13.1 (Pin_1), J14.1 (Pin_1), J15.1 (Pin_1), J16.1 (Pin_1), VoltReg1.2 (VO); no longer U2.190 (VDAC), U2.191 (3V3), U2.192 (3V3), U2.193 (3V3), U2.194 (3V3), U2.39 (GPIO_VDD), U2.40 (GPIO_VDD), U2.41 (GPIO_VDD), U2.42 (GPIO_VDD), U3.190 (VDAC), U3.191 (3V3), U3.192 (3V3), U3.193 (3V3), U3.194 (3V3), U3.39 (GPIO_VDD), U3.40 (GPIO_VDD), U3.41 (GPIO_VDD), U3.42 (GPIO_VDD), U4.190 (VDAC), U4.191 (3V3), U4.192 (3V3), U4.193 (3V3), U4.194 (3V3), U4.39 (GPIO_VDD), U4.40 (GPIO_VDD), U4.41 (GPIO_VDD), U4.42 (GPIO_VDD), U5.190 (VDAC), U5.191 (3V3), U5.192 (3V3), U5.193 (3V3), U5.194 (3V3), U5.39 (GPIO_VDD), U5.40 (GPIO_VDD), U5.41 (GPIO_VDD), U5.42 (GPIO_VDD)
- net +5V: now also J10.1 (Pin_1), J11.1 (Pin_1), J7.1 (Pin_1), J9.1 (Pin_1)
- net +BATT: now also C30.1, C30.1, J10.3 (Pin_3), J11.3 (Pin_3), L1.2, U7.6 (FB)
- net E_PIO16: no longer U2.184 (NC), U3.184 (NC), U4.184 (NC), U5.184 (NC)
- net E_PIO17: no longer U2.186 (NC), U3.186 (NC), U4.186 (NC), U5.186 (NC)
- net E_PIO19: no longer U2.183 (NC), U3.183 (NC), U4.183 (NC), U5.183 (NC)
- net E_PIO20: no longer U2.185 (NC), U3.185 (NC), U4.185 (NC), U5.185 (NC)
- net VCC: now also 1.8vReg1.2 (VO), C3.1
- net VDDSMPS: now also R9.2
- net at BAT1.1, C30.1, R6.1: now also C30.1, C30.1, C30.1, C30.1, C30.1, C30.1, C30.1, C30.1, R9.2, U6.2 (Input), U7.2 (Input); no longer BATCharge1.5 (BAT)
- net at U2.197 (VBAT), U2.198 (VBAT), U2.199 (VBAT)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: now also J7.2 (Pin_2)
- net at U3.197 (VBAT), U3.198 (VBAT), U3.199 (VBAT)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: now also J9.2 (Pin_2)
- net at U5.197 (VBAT), U5.198 (VBAT), U5.199 (VBAT)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: now also J11.2 (Pin_2)
- net at U4.197 (VBAT), U4.198 (VBAT), U4.199 (VBAT)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: now also J10.2 (Pin_2)
- net at MainMCU1.102 (VDD12DSI), MainMCU1.108 (VDD12DSI): now also R9.1
- net VSS: now reaches BAT1.2, C30.2, PowerMosfet2.3 (S2)
- net VSS: now also 1.8vReg1.1 (GND), Accel1.1 (CLKIN), Accel1.11 (FSYNC), Accel1.18 (GND), Alt1.2 (PS), Alt1.3 (GND), BATCharge1.1 (Temp), BATCharge1.1 (Temp), BATCharge1.3 (GND), BATCharge1.3 (GND), BatProt1.4 (VSS), BatProt1.4 (VSS), C10.2, C11.1, C12.2, C14.1, C14.2, C2.1, C2.1, C2.1, C2.1, C2.1, C2.1, C2.1, C2.1, C2.1, C2.1, C2.1, C2.2, C2.2, C2.2, C25.1, C29.1, C3.2, C3.2, C3.2, C30.2, C31.2, C32.2, C33.2, C34.2, C35.2, C36.2, C37.2, C38.2, C38.2, C39.2, C4.2, C40.2, C41.2, C41.2, C43.2, C44.2, C45.2, C46.2, C47.2, C5.2, C6.1, C6.2, C7.1, C8.1, C9.1, C9.1, D10.1 (A), D11.1 (A), D3.1 (A1), D3.1 (A1), D8.1 (A), D9.1 (A), D9.1 (A1), D9.1 (A1), GPS1.10 (GND), GPS1.12 (GND), GPS1.13 (GND), GPS1.2 (D_SEL), GPS1.24 (GND), IMU1.2 (SDX), IMU1.3 (SCX), IMU1.6 (GND), IMU1.7 (GND), J1.10 (gnd), J1.11 (gnd), J1.6 (VSS), J1.9 (SHIELD), J12.2 (Pin_2), J2.2 (Ext), J3.15, J3.S1 (SHIELD), J3.S2 (SHIELD), J4.10 (GND_1), J4.11 (GND_2), J4.12 (GND_3), J4.13 (GND_4), J4.6 (VSS), J4.9 (DET), J8.11, J8.17, J8.2, J8.5, J8.8, J8.SH, LoRaWan1.11 (GND), LoRaWan1.13 (GND), LoRaWan1.14 (GND), LoRaWan1.19 (GND), Magnetometer1.11 (VSS), Magnetometer1.9 (VSS), MainMCU1.100 (VSS), MainMCU1.105 (VSSDSI), MainMCU1.109 (VSSDSI), MainMCU1.112 (VSS), MainMCU1.119 (VSS), MainMCU1.12 (VSS), MainMCU1.134 (VSS), MainMCU1.137 (VSS), MainMCU1.14 (VSSSMPS), MainMCU1.151 (VSS), MainMCU1.159 (VSS), MainMCU1.173 (VSS), MainMCU1.24 (VSS), MainMCU1.38 (VSSA), MainMCU1.45 (VSS), MainMCU1.47 (VSS), MainMCU1.6 (VSS), MainMCU1.64 (VSS), MainMCU1.70 (VSS), MainMCU1.81 (VSS), MainMCU1.83 (VSS), MainMCU1.93 (VSS), P1.1 (P1), P1.10 (P10), P1.13 (P13), P1.16 (P16), P1.19 (P19), P1.4 (P4), P1.7 (P7), P2.1 (P1), P2.10 (P10), P2.13 (P13), P2.16 (P16), P2.19 (P19), P2.4 (P4), P2.7 (P7), P3.14 (P14), P3.20 (P20), P3.25 (P25), P3.30 (P30), P3.34 (P34), P3.39 (P39), P3.6 (P6), P3.9 (P9), P4.14 (P14), P4.20 (P20), P4.25 (P25), P4.30 (P30), P4.34 (P34), P4.39 (P39), P4.6 (P6), P4.9 (P9), PowerMosfet2.1 (S1), PowerMosfet2.1 (S1), Q1.1 (E), Q2.2 (S), Q3.2 (S), Q4.2 (S), R12.2, R15.2, R2.1, R2.1, R2.1, R2.1, R2.1, R2.1, R2.2, R22.1, R24.1, R26.2, R26.2, R3.1, R3.1, R6.1, R6.1, R7.2, R7.2, R8.2, R8.2, R9.2, R9.2, SW3.1, U2.1 (GND), U2.103 (GND), U2.104 (GND), U2.109 (GND), U2.110 (GND), U2.115 (GND), U2.116 (GND), U2.121 (GND), U2.122 (GND), U2.127 (GND), U2.13 (GND), U2.133 (GND), U2.134 (GND), U2.139 (GND), U2.14 (GND), U2.140 (GND), U2.145 (GND), U2.146 (GND), U2.151 (GND), U2.152 (GND), U2.157 (GND), U2.163 (GND), U2.164 (GND), U2.169 (GND), U2.170 (GND), U2.181 (GND), U2.182 (GND), U2.187 (GND), U2.188 (GND), U2.19 (GND), U2.195 (GND), U2.196 (GND), U2.20 (GND), U2.25 (GND), U2.26 (GND), U2.31 (GND), U2.32 (GND), U2.37 (GND), U2.38 (GND), U2.4 (GND), U2.43 (GND), U2.44 (GND), U2.49 (GND), U2.50 (GND), U2.55 (GND), U2.56 (GND), U2.61 (GND), U2.62 (GND), U2.67 (GND), U2.68 (GND), U2.7 (GND), U2.73 (GND), U2.74 (GND), U2.79 (GND), U2.8 (GND), U2.80 (GND), U2.85 (GND), U2.86 (GND), U2.91 (GND), U2.92 (GND), U2.97 (GND), U2.98 (GND), U3.1 (GND), U3.103 (GND), U3.104 (GND), U3.109 (GND), U3.110 (GND), U3.115 (GND), U3.116 (GND), U3.121 (GND), U3.122 (GND), U3.127 (GND), U3.13 (GND), U3.133 (GND), U3.134 (GND), U3.139 (GND), U3.14 (GND), U3.140 (GND), U3.145 (GND), U3.146 (GND), U3.151 (GND), U3.152 (GND), U3.157 (GND), U3.163 (GND), U3.164 (GND), U3.169 (GND), U3.170 (GND), U3.181 (GND), U3.182 (GND), U3.187 (GND), U3.188 (GND), U3.19 (GND), U3.195 (GND), U3.196 (GND), U3.20 (GND), U3.25 (GND), U3.26 (GND), U3.31 (GND), U3.32 (GND), U3.37 (GND), U3.38 (GND), U3.43 (GND), U3.44 (GND), U3.49 (GND), U3.50 (GND), U3.55 (GND), U3.56 (GND), U3.61 (GND), U3.62 (GND), U3.67 (GND), U3.68 (GND), U3.7 (GND), U3.73 (GND), U3.74 (GND), U3.79 (GND), U3.8 (GND), U3.80 (GND), U3.85 (GND), U3.86 (GND), U3.91 (GND), U3.92 (GND), U3.97 (GND), U3.98 (GND), U4.1 (GND), U4.103 (GND), U4.104 (GND), U4.109 (GND), U4.110 (GND), U4.115 (GND), U4.116 (GND), U4.121 (GND), U4.122 (GND), U4.127 (GND), U4.13 (GND), U4.133 (GND), U4.134 (GND), U4.139 (GND), U4.14 (GND), U4.140 (GND), U4.145 (GND), U4.146 (GND), U4.151 (GND), U4.152 (GND), U4.157 (GND), U4.163 (GND), U4.164 (GND), U4.169 (GND), U4.170 (GND), U4.181 (GND), U4.182 (GND), U4.187 (GND), U4.188 (GND), U4.19 (GND), U4.195 (GND), U4.196 (GND), U4.20 (GND), U4.25 (GND), U4.26 (GND), U4.31 (GND), U4.32 (GND), U4.37 (GND), U4.38 (GND), U4.43 (GND), U4.44 (GND), U4.49 (GND), U4.50 (GND), U4.55 (GND), U4.56 (GND), U4.61 (GND), U4.62 (GND), U4.67 (GND), U4.68 (GND), U4.7 (GND), U4.73 (GND), U4.74 (GND), U4.79 (GND), U4.8 (GND), U4.80 (GND), U4.85 (GND), U4.86 (GND), U4.91 (GND), U4.92 (GND), U4.97 (GND), U4.98 (GND), U5.1 (GND), U5.103 (GND), U5.104 (GND), U5.109 (GND), U5.110 (GND), U5.115 (GND), U5.116 (GND), U5.121 (GND), U5.122 (GND), U5.127 (GND), U5.13 (GND), U5.133 (GND), U5.134 (GND), U5.139 (GND), U5.14 (GND), U5.140 (GND), U5.145 (GND), U5.146 (GND), U5.151 (GND), U5.152 (GND), U5.157 (GND), U5.163 (GND), U5.164 (GND), U5.169 (GND), U5.170 (GND), U5.181 (GND), U5.182 (GND)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
- net power0 : now reaches U2.189 (VDAC)
- net power0 : now also U2.190 (VDAC), U2.191 (3V3), U2.192 (3V3), U2.193 (3V3), U2.194 (3V3), U2.39 (GPIO_VDD), U2.40 (GPIO_VDD), U2.41 (GPIO_VDD), U2.42 (GPIO_VDD), J14.2 (Pin_2)
- removed net GND: 1.8vReg1.1 (GND), Accel1.1 (CLKIN), Accel1.11 (FSYNC), Accel1.18 (GND), Alt1.2 (PS), Alt1.3 (GND), BATCharge1.1 (Temp), BATCharge1.1 (Temp), BATCharge1.3 (GND), BATCharge1.3 (GND), BatProt1.4 (VSS), BatProt1.4 (VSS), C10.2, C11.1, C12.2, C14.1, C14.2, C2.1, C2.1, C2.1, C2.1, C2.1, C2.1, C2.1, C2.1, C2.1, C2.1, C2.1, C2.2, C2.2, C2.2, C25.1, C29.1, C3.2, C3.2, C3.2, C30.2, C31.2, C32.2, C33.2, C34.2, C35.2, C36.2, C37.2, C38.2, C38.2, C39.2, C4.2, C40.2, C41.2, C41.2, C43.2, C44.2, C45.2, C46.2, C47.2, C5.2, C6.1, C6.2, C7.1, C8.1, C9.1, C9.1, D10.1 (A), D11.1 (A), D3.1 (A1), D3.1 (A1), D8.1 (A), D9.1 (A), D9.1 (A1), D9.1 (A1), GPS1.10 (GND), GPS1.12 (GND), GPS1.13 (GND), GPS1.2 (D_SEL), GPS1.24 (GND), IMU1.2 (SDX), IMU1.3 (SCX), IMU1.6 (GND), IMU1.7 (GND), J1.10 (gnd), J1.11 (gnd), J1.6 (VSS), J1.9 (SHIELD), J12.2 (Pin_2), J2.2 (Ext), J3.15, J3.S1 (SHIELD), J3.S2 (SHIELD), J4.10 (GND_1), J4.11 (GND_2), J4.12 (GND_3), J4.13 (GND_4), J4.6 (VSS), J4.9 (DET), J8.11, J8.17, J8.2, J8.5, J8.8, J8.SH, LoRaWan1.11 (GND), LoRaWan1.13 (GND), LoRaWan1.14 (GND), LoRaWan1.19 (GND), Magnetometer1.11 (VSS), Magnetometer1.9 (VSS), MainMCU1.100 (VSS), MainMCU1.105 (VSSDSI), MainMCU1.109 (VSSDSI), MainMCU1.112 (VSS), MainMCU1.119 (VSS), MainMCU1.12 (VSS), MainMCU1.134 (VSS), MainMCU1.137 (VSS), MainMCU1.14 (VSSSMPS), MainMCU1.151 (VSS), MainMCU1.159 (VSS), MainMCU1.173 (VSS), MainMCU1.24 (VSS), MainMCU1.38 (VSSA), MainMCU1.45 (VSS), MainMCU1.47 (VSS), MainMCU1.6 (VSS), MainMCU1.64 (VSS), MainMCU1.70 (VSS), MainMCU1.81 (VSS), MainMCU1.83 (VSS), MainMCU1.93 (VSS), P1.1 (P1), P1.10 (P10), P1.13 (P13), P1.16 (P16), P1.17 (P17), P1.19 (P19), P1.4 (P4), P1.7 (P7), P2.1 (P1), P2.10 (P10), P2.13 (P13), P2.16 (P16), P2.19 (P19), P2.4 (P4), P2.7 (P7), P3.14 (P14), P3.20 (P20), P3.25 (P25), P3.30 (P30), P3.34 (P34), P3.39 (P39), P3.6 (P6), P3.9 (P9), P4.14 (P14), P4.20 (P20), P4.25 (P25), P4.30 (P30), P4.34 (P34), P4.39 (P39), P4.6 (P6), P4.9 (P9), PowerMosfet2.1 (S1), PowerMosfet2.1 (S1), Q1.1 (E), Q2.2 (S), Q3.2 (S), Q4.2 (S), R12.2, R15.2, R2.1, R2.1, R2.1, R2.1, R2.1, R2.1, R2.2, R22.1, R24.1, R26.2, R26.2, R3.1, R3.1, R44.1, R6.1, R6.1, R7.2, R7.2, R8.2, R8.2, R9.2, R9.2, SW3.1, U2.1 (GND), U2.103 (GND), U2.104 (GND), U2.109 (GND), U2.110 (GND), U2.115 (GND), U2.116 (GND), U2.121 (GND), U2.122 (GND), U2.127 (GND), U2.13 (GND), U2.133 (GND), U2.134 (GND), U2.139 (GND), U2.14 (GND), U2.140 (GND), U2.145 (GND), U2.146 (GND), U2.151 (GND), U2.152 (GND), U2.157 (GND), U2.163 (GND), U2.164 (GND), U2.169 (GND), U2.170 (GND), U2.181 (GND), U2.182 (GND), U2.187 (GND), U2.188 (GND), U2.19 (GND), U2.195 (GND), U2.196 (GND), U2.20 (GND), U2.25 (GND), U2.26 (GND), U2.31 (GND), U2.32 (GND), U2.37 (GND), U2.38 (GND), U2.4 (GND), U2.43 (GND), U2.44 (GND), U2.49 (GND), U2.50 (GND), U2.55 (GND), U2.56 (GND), U2.61 (GND), U2.62 (GND), U2.67 (GND), U2.68 (GND), U2.7 (GND), U2.73 (GND), U2.74 (GND), U2.79 (GND), U2.8 (GND), U2.80 (GND), U2.85 (GND), U2.86 (GND), U2.88 (HDMI_HPD_N_1V8), U2.91 (GND), U2.92 (GND), U2.97 (GND), U2.98 (GND), U3.1 (GND), U3.103 (GND), U3.104 (GND), U3.109 (GND), U3.110 (GND), U3.115 (GND), U3.116 (GND), U3.121 (GND), U3.122 (GND), U3.127 (GND), U3.13 (GND), U3.133 (GND), U3.134 (GND), U3.139 (GND), U3.14 (GND), U3.140 (GND), U3.145 (GND), U3.146 (GND), U3.151 (GND), U3.152 (GND), U3.157 (GND), U3.163 (GND), U3.164 (GND), U3.169 (GND), U3.170 (GND), U3.181 (GND), U3.182 (GND), U3.187 (GND), U3.188 (GND), U3.19 (GND), U3.195 (GND), U3.196 (GND), U3.20 (GND), U3.25 (GND), U3.26 (GND), U3.31 (GND), U3.32 (GND), U3.36 (GPIO31), U3.37 (GND), U3.38 (GND), U3.43 (GND), U3.44 (GND), U3.49 (GND), U3.50 (GND), U3.55 (GND), U3.56 (GND), U3.61 (GND), U3.62 (GND), U3.67 (GND), U3.68 (GND), U3.7 (GND), U3.73 (GND), U3.74 (GND), U3.79 (GND), U3.8 (GND), U3.80 (GND), U3.85 (GND), U3.86 (GND), U3.88 (HDMI_HPD_N_1V8), U3.91 (GND), U3.92 (GND), U3.97 (GND), U3.98 (GND), U4.1 (GND), U4.103 (GND), U4.104 (GND), U4.109 (GND), U4.110 (GND), U4.115 (GND), U4.116 (GND), U4.121 (GND), U4.122 (GND), U4.127 (GND), U4.13 (GND), U4.133 (GND), U4.134 (GND), U4.139 (GND), U4.14 (GND), U4.140 (GND), U4.145 (GND), U4.146 (GND), U4.151 (GND), U4.152 (GND), U4.157 (GND), U4.163 (GND), U4.164 (GND), U4.169 (GND), U4.170 (GND), U4.181 (GND), U4.182 (GND), U4.187 (GND), U4.188 (GND), U4.19 (GND), U4.195 (GND), U4.196 (GND), U4.20 (GND), U4.25 (GND), U4.26 (GND), U4.31 (GND), U4.32 (GND), U4.37 (GND), U4.38 (GND), U4.43 (GND), U4.44 (GND), U4.49 (GND), U4.50 (GND), U4.55 (GND), U4.56 (GND), U4.61 (GND), U4.62 (GND), U4.67 (GND), U4.68 (GND), U4.7 (GND), U4.73 (GND), U4.74 (GND), U4.79 (GND), U4.8 (GND), U4.80 (GND), U4.85 (GND), U4.86 (GND), U4.88 (HDMI_HPD_N_1V8), U4.91 (GND), U4.92 (GND), U4.97 (GND), U4.98 (GND), U5.1 (GND), U5.103 (GND), U5.104 (GND), U5.109 (GND), U5.110 (GND), U5.115 (GND), U5.116 (GND), U5.121 (GND), U5.122 (GND), U5.127 (GND), U5.13 (GND), U5.133 (GND), U5.134 (GND), U5.139 (GND), U5.14 (GND), U5.140 (GND), U5.145 (GND), U5.146 (GND), U5.151 (GND), U5.152 (GND), U5.157 (GND)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
- new net: C30.1, U6.3 (CB)
- new net: C30.2, R7.2, U6.5 (VSW)
- new net: D17.3 (K), L1.1, U6.1 (Output)
- new net: C30.1, U6.7 (SS)
- new net: C30.2, R7.2, U7.5 (VSW)
- new net: D16.3 (K), L1.1, U7.1 (Output)
- new net: C30.1, U7.3 (CB)
- new net: C30.1, U7.7 (SS)
- new net: BATCharge1.5 (BAT), R9.1
- new net +5P: 1.8vReg1.3 (VI), C30.1, C30.1, J7.3 (Pin_3), J9.3 (Pin_3), L1.2, U6.6 (FB), VoltReg1.3 (VI)
- new net 1CAM1_IO0: P1.17 (P17), U3.36 (GPIO31)
- new net HDMI_HPD_N_1V8: R44.1, U2.88 (HDMI_HPD_N_1V8), U3.88 (HDMI_HPD_N_1V8), U4.88 (HDMI_HPD_N_1V8), U5.88 (HDMI_HPD_N_1V8)
- new net power1 : J13.2 (Pin_2), U3.190 (VDAC), U3.191 (3V3), U3.192 (3V3), U3.193 (3V3), U3.194 (3V3), U3.39 (GPIO_VDD), U3.40 (GPIO_VDD), U3.41 (GPIO_VDD), U3.42 (GPIO_VDD)
- new net power2 : J15.2 (Pin_2), U4.190 (VDAC), U4.191 (3V3), U4.192 (3V3), U4.193 (3V3), U4.194 (3V3), U4.39 (GPIO_VDD), U4.40 (GPIO_VDD), U4.41 (GPIO_VDD), U4.42 (GPIO_VDD)
- new net power3 : J16.2 (Pin_2), U5.190 (VDAC), U5.191 (3V3), U5.192 (3V3), U5.193 (3V3), U5.194 (3V3), U5.39 (GPIO_VDD), U5.40 (GPIO_VDD), U5.41 (GPIO_VDD), U5.42 (GPIO_VDD)
- no-connect marks 131 -> 135
