File: SDR_FlightComputer/KICAD Design Files/Sheet4.kicad_sch (KiCad schematic)
At the start: 109 parts, among them J13 502570-0893, SW1 SW_DIP_x02, U14 XC7Z010-1CLG400I, U15 MX25U1635EZNI-10G, U16 TXS02612RTWR, U17 RT9193-33B, U18 H5TQ4G63AFR, U19 MS5611-01BA, U21 BNO085, Y3 32.768kHz

Commit message: 1/10 Update 3
Connections:
- net PWR_Rx1 is gone; now on net PMOD7: U14.A14 (PS_MIO32_501)
- net PWR_Tx1 is gone; now on net PMOD3: U14.A16 (PS_MIO24_501)
- net PMOD3: no longer U14.C13 (PS_MIO29_501)
- net PMOD7: no longer U14.B13 (PS_MIO50_501)
Changed lines of the file:
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@@
-		)
-	)
-	(global_label "PWR_Rx1"
-		(shape bidirectional)
-		(at 715.01 219.075 0)
-		(fields_autoplaced yes)
-		(effects
-			(font
-				(size 1.27 1.27)
-			)
-			(justify left)
-		)
-		(property "Intersheetrefs" "${INTERSHEET_REFS}"
-			(at 727.5731 219.075 0)
-			(effects
-				(font
-					(size 1.27 1.27)
-				)
-				(justify left)
-				(hide yes)
-			)
 		)
 	)
@@
 		)
 	)
+	(global_label "PMOD3"
+		(shape bidirectional)
+		(at 715.01 198.755 0)
+		(fields_autoplaced yes)
+		(effects
+			(font
+				(size 1.27 1.27)
+			)
+			(justify left)
+		)
+		(property "Intersheetrefs" "${INTERSHEET_REFS}"
+			(at 725.6379 198.755 0)
+			(effects
+				(font
+					(size 1.27 1.27)
+				)
+				(justify left)
+				(hide yes)
+			)
+		)
+	)
 	(global_label "MAC_MDIO"
 		(shape bidirectional)
@@
 		(property "Intersheetrefs" "${INTERSHEET_REFS}"
 			(at 384.4426 313.055 0)
-			(effects
-				(font
-					(size 1.27 1.27)
-				)
-				(justify left)
-				(hide yes)
-			)
-		)
-	)
-	(global_label "PMOD3"
-		(shape bidirectional)
-		(at 715.01 112.395 0)
-		(fields_autoplaced yes)
-		(effects
-			(font
-				(size 1.27 1.27)
-			)
-			(justify left)
-		)
-		(property "Intersheetrefs" "${INTERSHEET_REFS}"
-			(at 725.6379 112.395 0)
 			(effects
 				(font
@@
 		)
 	)
-	(global_label "PWR_Tx1"
-		(shape bidirectional)
-		(at 715.01 198.755 0)
-		(fields_autoplaced yes)
-		(effects
-			(font
-				(size 1.27 1.27)
-			)
-			(justify left)
-		)
-		(property "Intersheetrefs" "${INTERSHEET_REFS}"
-			(at 727.2707 198.755 0)
-			(effects
-				(font
-					(size 1.27 1.27)
-				)
-				(justify left)
-				(hide yes)
-			)
-		)
-	)
 	(global_label "PS_MIO05_500_QSPI0_IO3"
 		(shape bidirectional)
@@
 		)
 	)
-	(global_label "PMOD7"
-		(shape bidirectional)
-		(at 715.01 163.195 0)
-		(fields_autoplaced yes)
-		(effects
-			(font
-				(size 1.27 1.27)
-			)
-			(justify left)
-		)
-		(property "Intersheetrefs" "${INTERSHEET_REFS}"
-			(at 725.6379 163.195 0)
-			(effects
-				(font
-					(size 1.27 1.27)
-				)
-				(justify left)
-				(hide yes)
-			)
-		)
-	)
 	(global_label "SDMMC_D0"
 		(shape bidirectional)
@@
 			(effects
 				(font
+					(size 1.27 1.27)
+				)
+				(justify left)
+				(hide yes)
+			)
+		)
+	)
+	(global_label "PMOD7"
+		(shape bidirectional)
+		(at 715.01 219.075 0)
+		(fields_autoplaced yes)
+		(effects
+			(font
+				(size 1.27 1.27)
+			)
+			(justify left)
+		)
+		(property "Intersheetrefs" "${INTERSHEET_REFS}"
+			(at 725.6379 219.075 0)
+			(effects
+				(font
