File: Main Flight Computer/KICAD Design Files/Sheet3.kicad_sch (KiCad schematic)
At the start: 73 parts, among them J10 RF2-49B-T-00-50-G-HDW, J11 RF2-49B-T-00-50-G-HDW, J12 RF2-49B-T-00-50-G-HDW, J8 73412-0110, J9 RF2-49B-T-00-50-G-HDW, T1 TCM1-63AX_, T2 TCM1-63AX_, T3 TCM1-63AX_, T4 TCM1-63AX_, U11 RT9193-33B, U12 AD9361BBCZ, U13 USB3320C-EZK-TR, Y2 25MHz

Commit message: 1/14 Update
Parts:
- U12: value AD9361BBCZ -> AD9363BBCZ
Changed lines of the file:
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@@
 			)
 		)
-		(property "Description" "\nAudio Transformers / Signal Transformers 1:1 CORE & WIRE Transformer, 10 - 6000 MHz, 50 ohms\n"
+		(property "Description" "Audio Transformers / Signal Transformers 1:1 CORE & WIRE Transformer, 10 - 6000 MHz, 50 ohms"
 			(at 316.865 92.71 0)
 			(effects
@@
 			)
 		)
-		(property "Description" "\nAudio Transformers / Signal Transformers 1:1 CORE & WIRE Transformer, 10 - 6000 MHz, 50 ohms\n"
+		(property "Description" "Audio Transformers / Signal Transformers 1:1 CORE & WIRE Transformer, 10 - 6000 MHz, 50 ohms"
 			(at 316.865 60.96 0)
 			(effects
@@
 			)
 		)
-		(property "Datasheet" " ~"
+		(property "Datasheet" "~"
 			(at 42.545 188.595 0)
 			(effects
@@
 			)
 		)
-		(property "Description" "\nAudio Transformers / Signal Transformers 1:1 CORE & WIRE Transformer, 10 - 6000 MHz, 50 ohms\n"
+		(property "Description" "Audio Transformers / Signal Transformers 1:1 CORE & WIRE Transformer, 10 - 6000 MHz, 50 ohms"
 			(at 316.865 28.575 0)
 			(effects
@@
 			)
 		)
-		(property "Value" "AD9361BBCZ"
+		(property "Value" "AD9363BBCZ"
 			(at 173.355 249.555 0)
 			(effects
@@
 			)
 		)
-		(property "Description" "\nRF Agile Transceiver\n"
+		(property "Description" "RF Agile Transceiver"
 			(at 187.96 148.59 0)
 			(effects
@@
 			)
 		)
-		(property "Description" "\nMicrochip USB3320C-EZK-TR, USB Transceiver, USB 2.0, 1.8 V, 3.3 V, 32-Pin QFN | Microchip Technology Inc. USB3320C-EZK-TR\n"
+		(property "Description" "Microchip USB3320C-EZK-TR, USB Transceiver, USB 2.0, 1.8 V, 3.3 V, 32-Pin QFN | Microchip Technology Inc. USB3320C-EZK-TR"
 			(at 328.93 185.42 0)
 			(effects
@@
 			)
 		)
-		(property "Description" "\n25 MHz ±10ppm Crystal 18pF 40 Ohms 4-SMD, No Lead\n"
+		(property "Description" "25 MHz ±10ppm Crystal 18pF 40 Ohms 4-SMD, No Lead"
 			(at 389.89 232.41 0)
 			(effects
@@
 			)
 		)
-		(property "Description" "\nAudio Transformers / Signal Transformers 1:1 CORE & WIRE Transformer, 10 - 6000 MHz, 50 ohms\n"
+		(property "Description" "Audio Transformers / Signal Transformers 1:1 CORE & WIRE Transformer, 10 - 6000 MHz, 50 ohms"
 			(at 320.04 128.27 0)
 			(effects
