File: Main Flight Computer/KICAD Design Files/IO_SDR_1.1.kicad_pcb (KiCad board)
At the start: 6 copper layers, 91.5 x 91.5 mm, 289 parts, among them J1 10118193-0001LF, J10 RF2-49B-T-00-50-G-HDW, J11 RF2-49B-T-00-50-G-HDW, J12 RF2-49B-T-00-50-G-HDW, J13 502570-0893, J2 10118193-0001LF, J3 Conn_01x03_Shielded, J4 Conn_02x20_Counter_Clockwise, J5 Conn_02x06_Odd_Even, J6 Conn_02x06_Odd_Even, J8 73412-0110, J9 RF2-49B-T-00-50-G-HDW, Q1 S8050, Q2 S8050, SW1 SW_DIP_x02, T1 TCM1-63AX_, T2 TCM1-63AX_, T3 TCM1-63AX_, T4 TCM1-63AX_, U1 TCMT1107, U11 RT9193-33B, U12 AD9363BBCZ, U13 USB3320C-EZK-TR, U14 XC7Z010-1CLG400I, U15 MX25U1635EZNI-10G, U16 TXS02612RTWR, U17 RT9193-33B, U18 H5TQ4G63AFR, U19 MS5611-01BA, U2 SY6280AAC, U21 BNO085, U3 AP3445W6-7, U4 AP3445W6-7, U5 TPS7A8101DRBT, U6 TPS7A8101DRBT, U7 AP3445W6-7, U8 AP3445W6-7, Y2 25MHz, Y3 32.768kHz

Commit message: 5/11 update
Parts:
- removed H101, H102, H103, H104: MountingHole_Pad, bac MicroMod Main Board v1:bac-PCB-Rail-Pad
- removed L2: R0603, Inductor_SMD:L_0603_1608Metric_Pad1.05x0.95mm_HandSolder
Connections:
- U14 pad J10: +1V8 -> GND
Routing:
- net +1V8: track 77.2 -> 76.7 mm, vias 63 -> 77
- net GND: track 279.7 -> 280.1 mm, vias 378 -> 380
Other:
- board text removed: "BOOTSEL"
- board text removed: "RESET"
- board text removed: "envious.design"
