File: Main Flight Computer/KICAD Design Files/Sheet1.kicad_sch (KiCad schematic)
At the start: 103 parts, among them J1 10118193-0001LF, J2 10118193-0001LF, J3 Conn_01x03_Shielded, J4 Conn_02x20_Counter_Clockwise, J5 Conn_02x06_Odd_Even, J6 Conn_02x06_Odd_Even, Q1 S8050, Q2 S8050, U1 TCMT1107, U2 SY6280AAC, U3 TCS4615, U4 TCS4615, U5 TPS7A8101DRBT, U6 TPS7A8101DRBT, U7 TCS4615, U8 TCS4615

Commit message: 1/14 Update
Parts:
- QA1, QA2, QA3: value HR8031GS6 -> SQ2361ES
- U3, U4, U7, U8: value TCS4615 -> AP3445W6-7
Other:
- note added: "JTAG PINS"
- note removed: "JATG PINS"
Changed lines of the file:
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@@
 		)
 	)
-	(text "JATG PINS\n "
+	(text "JTAG PINS\n "
 		(exclude_from_sim no)
 		(at 234.95 230.505 0)
@@
 			)
 		)
-		(property "Value" "HR8031GS6"
+		(property "Value" "SQ2361ES"
 			(at 95.885 187.325 90)
 			(effects
@@
 			)
 		)
-		(property "Value" "TCS4615"
+		(property "Value" "AP3445W6-7"
 			(at 338.2772 164.0078 0)
 			(effects
@@
 			)
 		)
-		(property "Value" "TCS4615"
+		(property "Value" "AP3445W6-7"
 			(at 339.0646 109.2708 0)
 			(effects
@@
 			)
 		)
-		(property "Value" "TCS4615"
+		(property "Value" "AP3445W6-7"
 			(at 169.545 135.001 0)
 			(effects
@@
 			)
 		)
-		(property "Value" "HR8031GS6"
+		(property "Value" "SQ2361ES"
 			(at 84.455 108.585 0)
 			(effects
@@
 			)
 		)
-		(property "Value" "HR8031GS6"
+		(property "Value" "SQ2361ES"
 			(at 70.485 109.22 0)
 			(effects
@@
 			)
 		)
-		(property "Value" "TCS4615"
+		(property "Value" "AP3445W6-7"
 			(at 207.645 57.531 0)
 			(effects

Commit message: 1/14 2nd update
Parts:
- C4: footprint Capacitor_SMD:C_0805_2012Metric_Pad1.18x1.45mm_HandSolder -> Capacitor_SMD:C_1206_3216Metric_Pad1.33x1.80mm_HandSolder

Commit message: 5/11 update
Parts:
- removed L2: R0603, Inductor_SMD:L_0603_1608Metric_Pad1.05x0.95mm_HandSolder, symbol Device:L_Iron
Changed lines of the file:
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@@
-	)
-	(symbol
-		(lib_id "Device:L_Iron")
-		(at 219.71 113.411 90)
-		(unit 1)
-		(exclude_from_sim no)
-		(in_bom yes)
-		(on_board yes)
-		(dnp no)
-		(property "Reference" "L2"
-			(at 219.202 110.617 90)
-			(effects
-				(font
-					(size 1.27 1.27)
-				)
-			)
-		)
-		(property "Value" "R0603"
-			(at 219.075 115.316 90)
-			(effects
-				(font
-					(size 1.27 1.27)
-				)
-			)
-		)
-		(property "Footprint" "Inductor_SMD:L_0603_1608Metric_Pad1.05x0.95mm_HandSolder"
-			(at 219.71 113.411 0)
-			(effects
-				(font
-					(size 1.27 1.27)
-				)
-				(hide yes)
-			)
-		)
-		(property "Datasheet" "~"
-			(at 219.71 113.411 0)
-			(effects
-				(font
-					(size 1.27 1.27)
-				)
-				(hide yes)
-			)
-		)
-		(property "Description" ""
-			(at 219.71 113.411 0)
-			(effects
-				(font
-					(size 1.27 1.27)
-				)
-				(hide yes)
-			)
-		)
-		(property "JLCPCB Part#" ""
-			(at 219.71 113.411 0)
-			(effects
-				(font
-					(size 1.27 1.27)
-				)
-				(hide yes)
-			)
-		)
-		(pin "1"
-		)
-		(pin "2"
-		)
-		(instances
-			(project "IO_SDR_1.1"
-				(path "/38786148-0fd1-46d3-8412-9a7876291ebf/b3b43e8b-7f47-4b04-880b-01695a760090"
-					(reference "L2")
-					(unit 1)
-				)
-			)
-		)
 	)
 	(symbol
