File: Main Flight Computer/KICAD Design Files/Sheet4.kicad_sch (KiCad schematic)
At the start: 109 parts, among them J13 502570-0893, SW1 SW_DIP_x02, U14 XC7Z010-1CLG400I, U15 MX25U1635EZNI-10G, U16 TXS02612RTWR, U17 RT9193-33B, U18 H5TQ4G63AFR, U19 MS5611-01BA, U21 BNO085, Y3 32.768kHz

Commit message: 5/11 update
Connections:
- net +1V8: no longer U14.J10 (GNDADC_0)
- net GND: now also U14.J10 (GNDADC_0)
Changed lines of the file:
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@@
 	(paper "A1")
 	(junction
-		(at 577.85 185.42)
-		(diameter 0)
-		(color 0 0 0 0)
-	)
-	(junction
 		(at 608.2284 361.0102)
 		(diameter 0)
@@
 	)
 	(no_connect
-		(at 565.785 190.5)
+		(at 565.404 190.5)
 	)
 	(no_connect
@@
 	(wire
 		(pts
-			(xy 565.404 185.42) (xy 577.85 185.42)
-		)
-		(stroke
-			(width 0)
-			(type default)
-		)
-	)
-	(wire
-		(pts
 			(xy 707.39 60.96) (xy 714.375 60.96)
 		)
@@
 	(wire
 		(pts
-			(xy 577.85 185.42) (xy 577.85 180.34)
+			(xy 577.85 180.34) (xy 577.85 195.58)
 		)
 		(stroke
@@
 	(wire
 		(pts
-			(xy 577.85 185.42) (xy 577.85 195.58)
-		)
-		(stroke
-			(width 0)
-			(type default)
-		)
-	)
-	(wire
-		(pts
 			(xy 720.4964 404.6474) (xy 725.5764 404.6474)
 		)
@@
 					(unit 1)
 				)
+			)
+		)
+	)
+	(symbol
+		(lib_name "GND_1")
+		(lib_id "power:GND")
+		(at 565.404 185.42 90)
+		(unit 1)
+		(exclude_from_sim no)
+		(in_bom yes)
+		(on_board yes)
+		(dnp no)
+		(property "Reference" "#PWR094"
+			(at 571.754 185.42 0)
+			(effects
+				(font
+					(size 1.27 1.27)
+				)
+				(hide yes)
+			)
+		)
+		(property "Value" "GND"
+			(at 570.484 185.42 90)
+			(effects
+				(font
+					(size 1.27 1.27)
+				)
+			)
+		)
+		(property "Footprint" ""
+			(at 565.404 185.42 0)
+			(effects
+				(font
+					(size 1.27 1.27)
+				)
+				(hide yes)
+			)
+		)
+		(property "Datasheet" "~"
+			(at 565.404 185.42 0)
+			(effects
+				(font
+					(size 1.27 1.27)
+				)
+				(hide yes)
+			)
+		)
+		(property "Description" ""
+			(at 565.404 185.42 0)
+			(effects
+				(font
+					(size 1.27 1.27)
+				)
+				(hide yes)
+			)
+		)
+		(pin "1"
+		)
+		(instances
+			(project "IO_SDR_1.1"
+				(path "/38786148-0fd1-46d3-8412-9a7876291ebf/643e53b8-38bd-42e3-86de-6cc8c6c09224"
+					(reference "#PWR094")
+					(unit 1)
+				)
